Commit message: feat: modularize JAKA keyboard control and synchronize tool frames
Move keyboard entrypoints and YAML into the application package, split control
responsibilities, and add asynchronous cycle logging with offline analysis.
Use explicit positive enable switches and preserve a frozen original baseline.
Synchronize JAKA URDF/MJCF tool frames and link masses with the reference model.

Validation: 223 offline tests passed; two pre-existing planning import errors
were excluded. Command-trace, logging and boolean configuration checks passed.
No real-hardware run was performed.

File: simulation/mujoco/models/jaka/urdf/tracer_jaka_zu5.urdf (robot description, URDF)
Before this commit: robot tracer_jaka_zu5, 34 links, 33 joints
Links:
- link Link_0: mass 1.0392 -> 0.905
- link Link_1: mass 1.5135 -> 2.877
- link Link_2: mass 1.5847 -> 7.293
- link Link_3: mass 1.8069 -> 1.707
- link Link_4: mass 1.5525 -> 1.184
- link Link_5: mass 1.3339 -> 1.228
- link Link_6: mass 1.4169 -> 0.289
Joints:
- joint tool0_joint: origin xyz=0 0 0.27 rpy=0 0 0 -> xyz=0 0 0.27 rpy=0 0 3.141592653589793

Commit message: add logs and joy

File: simulation/mujoco/models/jaka/urdf/tracer_jaka_zu5.urdf (robot description, URDF)
Before this commit: robot tracer_jaka_zu5, 34 links, 33 joints
Joints:
- joint tool0_joint: origin xyz=0 0 0.27 rpy=0 0 3.141592653589793 -> xyz=0 0 0.195 rpy=0 0 3.141592653589793
